Commit message: Integrating the oakd sensor and ensuring a compatible ros/gazebo environment

File: sjtu_drone_description/urdf/sjtu_drone.urdf (robot description, URDF)
Before this commit: robot sjtu_drone, 5 links, 4 joints
Links:
- added link oakd_lite_link, mass 0.061; collision box size=0.04 0.09 0.025; visual mesh filename=file:///ros2_ws/install/sjtu_drone_description/share/sjtu_d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
- link base_link: geometry collision mesh filename=file:///ros2_ws/install/sjtu_drone_description/share/sjtu_d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; visual mesh filename=file:///ros2_ws/install/sjtu_drone_description/share/sjtu_d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
Joints:
- added joint oakd_lite_joint: type fixed, parent base_link, child oakd_lite_link, origin xyz=0.25 0 0 rpy=0 0 0

File: sjtu_drone_description/urdf/sjtu_drone.urdf.xacro (robot description, xacro)
@@ -54,18 +54,29 @@
   </joint>
   <link name="bottom_cam_link"/>
-    <!-- OakD-Lite Camera Link -->
-  <link name="oakd_lite_link">
+  <!-- OakD-Lite link -->
+   <link name="oakd_lite_link">
     <visual>
+      <origin xyz="0 0 0" rpy="0 0 0"/>
       <geometry>
-        <mesh filename="model://OakD-Lite/meshes/OAK-D_LITE_V1.dae" scale="0.001 0.001 0.001"/>
+        <mesh filename="file://$(find sjtu_drone_description)/models/OakD-Lite/meshes/OakDLite.dae"/>
       </geometry>
+    </visual>
+    <collision>
       <origin xyz="0 0 0" rpy="0 0 0"/>
-    </visual>
+      <geometry>
+        <box size="0.04 0.09 0.025"/>
+      </geometry>
+    </collision>
+    <inertial>
+      <mass value="0.061"/>
+      <origin xyz="0 0 0" rpy="0 0 0"/>
+      <inertia ixx="0.0001" ixy="0" ixz="0" iyy="0.0001" iyz="0" izz="0.0001"/>
+    </inertial>
   </link>
-  <!-- Fixed joint to attach OakD-Lite to the base of the drone -->
+  <!-- Fixed joint from base_link -->
   <joint name="oakd_lite_joint" type="fixed">
     <parent link="base_link"/>
     <child link="oakd_lite_link"/>
-    <origin xyz="0.05 0 0.03" rpy="0 0 0"/>
+    <origin xyz="0.25 0 0" rpy="0 0 0"/>
   </joint>
   <gazebo>
@@ -254,31 +265,59 @@
     </sensor>
   </gazebo>
-  <!--OakD-Lite stero depth sensing camera-->
-  <gazebo reference="oakd_lite_link">
-    <sensor name="oakd_camera" type="depth">
-      <always_on>true</always_on>
+  <!--OAKD-LITE REFERENCE-->
+ <gazebo reference="oakd_lite_link">
+    <sensor name="oakd_rgb_camera_sensor" type="camera">
+      <pose>0.01233 -0.03 0.01878 0 0 0</pose>
+      <always_on>1</always_on>
       <visualize>true</visualize>
-      <update_rate>30.0</update_rate>
-      <camera>
-        <horizontal_fov>1.3962634</horizontal_fov>
+      <update_rate>30</update_rate>
+      <camera name="IMX214">
+        <horizontal_fov>1.204</horizontal_fov>
         <image>
-          <width>640</width>
-          <height>480</height>
+          <width>1920</width>
+          <height>1080</height>
           <format>R8G8B8</format>
         </image>
         <clip>
           <near>0.1</near>
-          <far>10.0</far>
+          <far>100</far>
         </clip>
       </camera>
-      <plugin name="oakd_camera_plugin" filename="libgazebo_ros_depth_camera.so">
-        <camera_name>oakd_camera</camera_name>
-        <image_topic_name>image_raw</image_topic_name>
-        <depth_image_topic_name>depth/image_raw</depth_image_topic_name>
-        <camera_info_topic_name>camera_info</camera_info_topic_name>
+      <plugin name="oakd_rgb_camera_controller" filename="libgazebo_ros_camera.so">
+        <ros>
+          <namespace>${mp['namespace']}</namespace>
+          <remapping>image_raw:=oakd/rgb/image_raw</remapping>
+          <remapping>camera_info:=oakd/rgb/camera_info</remapping>
+        </ros>
         <frame_name>oakd_lite_link</frame_name>
-        <ros>
-          <namespace>${mp['namespace']}</namespace>
-        </ros>
+      </plugin>
+    </sensor>
+    <sensor name="oakd_depth_camera_sensor" type="depth">
+      <pose>0.01233 -0.03 0.01878 0 0 0</pose>
+      <always_on>1</always_on>
+      <visualize>true</visualize>
+      <update_rate>30</update_rate>
+      <camera name="StereoOV7251">
+        <horizontal_fov>1.274</horizontal_fov>
+        <image>
+          <width>640</width>
+          <height>480</height>
+          <format>R_FLOAT32</format>
+        </image>
+        <clip>
+          <near>0.2</near>
+          <far>19.1</far>
+        </clip>
+      </camera>
+      <plugin name="oakd_depth_camera_controller" filename="libgazebo_ros_depth_camera.so">
+        <ros>
+          <namespace>${mp['namespace']}</namespace>
+          <remapping>image_raw:=oakd/depth/image_raw</remapping>
+          <remapping>camera_info:=oakd/depth/camera_info</remapping>
+          <remapping>points:=oakd/depth/points</remapping>
+        </ros>
+        <frame_name>oakd_lite_link</frame_name>
+        <point_cloud_cutoff>0.2</point_cloud_cutoff>
+        <point_cloud_cutoff_max>19.1</point_cloud_cutoff_max>
       </plugin>
     </sensor>
